File: schemas/circuit_diagram_03/circuit_diagram.sch (KiCad schematic (older format))
At the start: 75 parts, among them J1 Conn_01x02_Male, M1 PUMP_Motor, M2 Motor_DC, M3 Motor_DC, M4 Motor_DC, Q1 Q_NMOS_DGS, Q2 Q_Photo_NPN, Q3 Q_Photo_NPN, Q4 Q_Photo_NPN, Q5 Q_Photo_NPN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

Commit message: Web communication fixed
Parts:
- removed R1, R2, R22, R3, R4, R41, R43, R5, R6, R7: R, Resistor_SMD:R_0805_2012Metric_Pad1.15x1.40mm_HandSolder, symbol Device:R
- R10, R11, R12, R13, R14, R31, R42, R44, R8, R9: value R -> 2K
- R15, R17, R18, R19, R20, R21, R23, R24, R25, R26, R27, R28, R29, R30, R32: value R -> 300
Connections:
- net +5V: no longer R19.2, R20.2, R21.2
- net at U1.11 (D0): now also Q2.2 (E), R8.1
- net at U1.12 (D1): now also Q3.2 (E), R9.1
- net at U1.13 (D2): now also Q4.2 (E), R10.1
- net at U1.14 (D3): now also Q5.2 (E), R11.1
- net at U1.3 (D4): now also Q6.2 (E), R12.1
- net at U1.4 (D5): now also Q7.2 (E), R13.1
- net at U1.5 (D6): now also Q8.2 (E), R14.1
- net at U1.6 (D7): now also R42.2, SW1.3
- net at R31.2, U19.3: now also U22.11 (D0)
- net at U22.12 (D1): now also R44.2, SW2.3
- new net: R19.2, R20.2, R21.2
Other:
- moved on the sheet: Q6, Q7, Q8, R12, R13, R14, R19, R20, R21
